File: rcnet.sch (KiCad schematic (older format))
At the start: 40 parts, among them IC1 LM1117, IC2 ATMEGA2560-A, P1 UART2, P2 UART1, P3 FTDI, P4 CONN_5, P5 I2C, P6 ICSP, P7 MOTEURS, P8 RX, Q1 2N7002, Q2 2N7002, U1 MS5611, U2 HMC5883L, U3 MPU6050, X1 16MHz

Commit message: Add V2
Parts:
- removed C3, C5: 10µF, symbol CAPAPOL
- removed C7: 4.7µF, symbol CAPAPOL
- removed IC1: LM1117, symbol LM1117
- removed P1: UART2, symbol CONN_4
- removed P2: UART1, symbol CONN_4
- removed P4: CONN_5, symbol CONN_5
- removed P8: RX, symbol CONN_8
- removed U2: HMC5883L, symbol HMC5883L
- added C3, C5: 1µF, symbol C
- added C7: 0.1µF, symbol C
- added D4, D5: LED, symbol LED
- added F1: FUSE, symbol FUSE
- added IC1: MCP1702, symbol MCP1702
- added K1: CAM, symbol CONN_3
- added P1: UARTS, symbol CONN_6
- added P11: MOTEURSGND, symbol CONN_8
- added P12: MOTEURS5V, symbol CONN_8
- added P13, P14: CONN_2, symbol CONN_2
- added P3: AUX, symbol CONN_5
- added P7: RX, symbol CONN_10
- added P8: LIPO, symbol CONN_2
- added P9: EXTENTION, symbol CONN_6
- added R10: 32.4k, symbol R
- added R11, R12: 320, symbol R
- added R13, R14, R15, R16, R17, R18, R19, R20, R21, R22, R23, R24, R25, R26, R27, R29, R30, R31, R32, R33, R34, R35, R36, R37, R38: 2k, symbol R
- added R28: 10k, symbol R
- added R9: 76.8k, symbol R
- added RSSI1: CONN_1, symbol CONN_1
- C2, C4: value C -> 22pF
- C8: value 0.22µF -> 0.1µF
- renumbered P3 to P2, P5 to P4, P6 to P5, P7 to P6
Connections:
- net labels added: +BATT, C_PITCH, C_ROLL, C_TRIG, F5V, GNDP, MAG_CL, MAG_DA, MPU_INT, RSSI, RXD2, RXD3, STATUS, TXD2, TXD3
- wire segments 158 -> 211
- no-connect marks 61 -> 46
Other:
- moved on the sheet: D3, P2, P5, R8
